File: Caution_SAO/Caution_SAO.kicad_pcb (KiCad board)
At the start: 2 copper layers, 40 x 40 mm, 5 parts, among them J1 Conn_02x03_Counter_Clockwise

Commit message: Working on the main village base badge
Parts:
- added svg2mod: G***, Images:master_caution, F.Cu at (119.0, 118.6)
- moved R2 15.6 mm to (107.7, 135.9), turned to 0 degrees
- moved J1 14.0 mm to (116.8, 133.3)
- moved R1 10.4 mm to (108.0, 129.5), turned to 0 degrees
Routing:
- net Net-(D1-Pad2): track 8.10 -> 13.2 mm
- net VCC: track 15.3 -> 13.4 mm
- net Net-(D2-Pad2): track 32.1 -> 30.4 mm
Other:
- net class Default removed
- board text added: "@cybertestpilot"
- board text removed: "MASTER CAUTION"
