File: Warning_SAO/Master_Warning.kicad_pcb (KiCad board)
At the start: 2 copper layers, 39.9 x 14.9 mm, 6 parts, among them J1 Conn_02x03_Counter_Clockwise

Commit message: updated per latest protoype discoveries
Parts:
- moved R1 22.0 mm to (209.4, 86.5), turned to -90 degrees
- moved R2 18.6 mm to (212.6, 86.4), turned to -90 degrees
- moved J1 1.01 mm to (227.1, 85.1)
Connections:
- J1 pad 5: unconnected-(J1-Pad5) -> Net-(J1-Pad1)
Routing:
- net Net-(J1-Pad1): track 14.6 -> 58.4 mm
- net Net-(D1-Pad2): track 25.3 -> 4.92 mm
- net Net-(D2-Pad2): track 18.9 -> 4.35 mm
Other:
- board text added: "Aerospace Village v03"
- board text added: "Alt. GPIO1"
- board text removed: "aerospace village v02"
