File: Warning_SAO/Master_Warning.kicad_sch (KiCad schematic)
At the start: 5 parts

Commit message: updated per latest protoype discoveries
Parts:
- D1, D2: value (none) -> LED; footprint (none) -> sunled:XZM2CRK45WT-9
- J1: value (none) -> Conn_02x03_Counter_Clockwise; footprint (none) -> Connector_PinHeader_2.54mm:PinHeader_2x03_P2.54mm_Vertical
- R1: value (none) -> 330; footprint (none) -> Resistor_SMD:R_1206_3216Metric
- R2: value (none) -> 300; footprint (none) -> Resistor_SMD:R_1206_3216Metric
Connections:
- net at J1.1 (Pin_1), R1.2, R2.2: now also J1.5 (Pin_5)
- no-connect marks 4 -> 3
Changed lines of the file:
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@@
   (junction (at 161.29 104.14) (diameter 0) (color 0 0 0 0)
+  )
+  (junction (at 161.29 105.41) (diameter 0) (color 0 0 0 0)
   )
   (junction (at 128.27 100.33) (diameter 0) (color 0 0 0 0)
@@
   (no_connect (at 142.24 100.33))
   (no_connect (at 142.24 105.41))
-  (no_connect (at 142.24 102.87))
   (no_connect (at 129.54 105.41))
+  (wire (pts (xy 149.86 102.87) (xy 149.86 107.95))
+    (stroke (width 0) (type default) (color 0 0 0 0))
+  )
+  (wire (pts (xy 161.29 105.41) (xy 161.29 107.95))
+    (stroke (width 0) (type default) (color 0 0 0 0))
+  )
   (wire (pts (xy 128.27 95.25) (xy 153.67 95.25))
     (stroke (width 0) (type default) (color 0 0 0 0))
   )
+  (wire (pts (xy 149.86 107.95) (xy 161.29 107.95))
+    (stroke (width 0) (type default) (color 0 0 0 0))
+  )
   (wire (pts (xy 157.48 86.36) (xy 157.48 83.82))
     (stroke (width 0) (type default) (color 0 0 0 0))
@@
     (stroke (width 0) (type default) (color 0 0 0 0))
   )
-  (wire (pts (xy 161.29 105.41) (xy 161.29 104.14))
+  (wire (pts (xy 161.29 104.14) (xy 161.29 105.41))
     (stroke (width 0) (type default) (color 0 0 0 0))
   )
@@
     (stroke (width 0) (type default) (color 0 0 0 0))
   )
+  (wire (pts (xy 142.24 102.87) (xy 149.86 102.87))
+    (stroke (width 0) (type default) (color 0 0 0 0))
+  )
   (wire (pts (xy 157.48 96.52) (xy 157.48 93.98))
     (stroke (width 0) (type default) (color 0 0 0 0))
@@
     (in_bom yes) (on_board yes)
     (property "Reference" "J1" (id 0) (at 135.89 94.8182 0))
-    (property "Value" "" (id 1) (at 135.89 97.1296 0))
-    (property "Footprint" "" (id 2) (at 134.62 102.87 0)
+    (property "Value" "Conn_02x03_Counter_Clockwise" (id 1) (at 135.89 97.1296 0))
+    (property "Footprint" "Connector_PinHeader_2.54mm:PinHeader_2x03_P2.54mm_Vertical" (id 2) (at 134.62 102.87 0)
       (effects (font (size 1.27 1.27)) hide)
     )
@@
       (effects (font (size 1.27 1.27)) (justify left))
     )
-    (property "Value" "" (id 1) (at 159.512 91.1352 90)
-      (effects (font (size 1.27 1.27)) (justify left))
-    )
-    (property "Footprint" "" (id 2) (at 157.48 90.17 0)
+    (property "Value" "LED" (id 1) (at 159.512 91.1352 90)
+      (effects (font (size 1.27 1.27)) (justify left))
+    )
+    (property "Footprint" "sunled:XZM2CRK45WT-9" (id 2) (at 157.48 90.17 0)
       (effects (font (size 1.27 1.27)) hide)
     )
@@
       (effects (font (size 1.27 1.27)) (justify left))
     )
-    (property "Value" "" (id 1) (at 167.132 91.1352 90)
-      (effects (font (size 1.27 1.27)) (justify left))
-    )
-    (property "Footprint" "" (id 2) (at 165.1 90.17 0)
+    (property "Value" "LED" (id 1) (at 167.132 91.1352 90)
+      (effects (font (size 1.27 1.27)) (justify left))
+    )
+    (property "Footprint" "sunled:XZM2CRK45WT-9" (id 2) (at 165.1 90.17 0)
       (effects (font (size 1.27 1.27)) hide)
     )
@@
       (effects (font (size 1.27 1.27)) (justify left))
     )
-    (property "Value" "" (id 1) (at 159.258 101.473 0)
-      (effects (font (size 1.27 1.27)) (justify left))
-    )
-    (property "Footprint" "" (id 2) (at 155.702 100.33 90)
+    (property "Value" "330" (id 1) (at 159.258 101.473 0)
+      (effects (font (size 1.27 1.27)) (justify left))
+    )
+    (property "Footprint" "Resistor_SMD:R_1206_3216Metric" (id 2) (at 155.702 100.33 90)
       (effects (font (size 1.27 1.27)) hide)
     )
@@
       (effects (font (size 1.27 1.27)) (justify left))
     )
-    (property "Value" "" (id 1) (at 166.878 101.473 0)
-      (effects (font (size 1.27 1.27)) (justify left))
-    )
-    (property "Footprint" "" (id 2) (at 163.322 100.33 90)
+    (property "Value" "300" (id 1) (at 166.878 101.473 0)
+      (effects (font (size 1.27 1.27)) (justify left))
+    )
+    (property "Footprint" "Resistor_SMD:R_1206_3216Metric" (id 2) (at 163.322 100.33 90)
       (effects (font (size 1.27 1.27)) hide)
     )
@@
       (effects (font (size 1.27 1.27)) hide)
     )
-    (property "Value" "" (id 1) (at 122.5042 100.33 90)
+    (property "Value" "PWR_FLAG" (id 1) (at 122.5042 100.33 90)
       (effects (font (size 1.27 1.27)) (justify left))
     )
@@
       (effects (font (size 1.27 1.27)) hide)
     )
-    (property "Value" "" (id 1) (at 122.4788 102.997 90)
+    (property "Value" "GND" (id 1) (at 122.4788 102.997 90)
       (effects (font (size 1.27 1.27)) (justify right))
     )
@@
       (effects (font (size 1.27 1.27)) hide)
     )
-    (property "Value" "" (id 1) (at 157.353 79.4258 0))
+    (property "Value" "GND" (id 1) (at 157.353 79.4258 0))
     (property "Footprint" "" (id 2) (at 157.48 83.82 0)
       (effects (font (size 1.27 1.27)) hide)
@@
       (effects (font (size 1.27 1.27)) hide)
     )
-    (property "Value" "" (id 1) (at 164.973 79.4258 0))
+    (property "Value" "GND" (id 1) (at 164.973 79.4258 0))
     (property "Footprint" "" (id 2) (at 165.1 83.82 0)
       (effects (font (size 1.27 1.27)) hide)
