File: gold_star_SAO/gold_star.kicad_pcb (KiCad board)
At the start: 2 copper layers, 38.3 x 37.8 mm, 2 parts, among them J1 Conn_02x03_Counter_Clockwise

Commit message: Small update to basic gold star
Other:
- board text added: "@av_pubs"
- board text removed: "@pubs"
Changed lines of the file:
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@@
     (pad_to_mask_clearance 0)
     (pcbplotparams
-      (layerselection 0x00000fc_ffffffff)
+      (layerselection 0x00010fc_ffffffff)
       (disableapertmacros false)
       (usegerberextensions true)
@@
     (effects (font (size 1 1) (thickness 0.15)) (justify mirror))
   )
-  (gr_text "@pubs" (at 127 63.5) (layer "B.SilkS")
+  (gr_text "@av_pubs" (at 127 68.58) (layer "B.SilkS")
     (effects (font (size 1 1) (thickness 0.15)) (justify mirror))
   )
