File: gold_star_v2_SAO/gold_star_v2_SAO.kicad_pcb (KiCad board)
At the start: 2 copper layers, 38.3 x 37.8 mm, 2 parts, among them J1 Conn_02x03_Counter_Clockwise

Commit message: v0.1 of the gold star with copper showing
Parts:
- removed the G*** at (127.0, 66.0)
- added G*** (x2): LOGO, LOGO, F.Cu at (127.0, 66.0)
Routing:
- added copper zone on F.Cu, net (none)
Other:
- board text added: "@av_pubs"
- board text removed: "@pubs"
