File: 787 with Boeing logo SAO extender/787.kicad_sch (KiCad schematic)
At the start: 0 parts

Commit message: added schematic to 787 SAO extender
Parts:
- added D: LED, symbol Device:LED
- added J (x3): Conn_02x03_Counter_Clockwise, symbol Connector_Generic:Conn_02x03_Counter_Clockwise
- added R: R, symbol Device:R
Connections:
- new net: J.3 (Pin_3), J.3 (Pin_3), J.3 (Pin_3)
- new net: J.4 (Pin_4), J.4 (Pin_4), J.4 (Pin_4)
- new net: J.5 (Pin_5), J.5 (Pin_5), J.5 (Pin_5)
- new net: J.6 (Pin_6), J.6 (Pin_6), J.6 (Pin_6)
- new net: D.2 (A), R.1
- new net +3V3: J.1 (Pin_1), J.1 (Pin_1), J.1 (Pin_1), R.2
- new net GND: D.1 (K), J.2 (Pin_2), J.2 (Pin_2), J.2 (Pin_2)
