File: B2/B2.kicad_sch (KiCad schematic)
At the start: 0 parts

Commit message: b2 with schematic and green led
Parts:
- added D: LED, symbol Device:LED
- added J: Conn_02x03_Odd_Even, symbol Connector_Generic:Conn_02x03_Odd_Even
- added R: R, symbol Device:R
Connections:
- new net: J.1 (Pin_1), R.2
- new net: D.2 (A), R.1
- new net GND: D.1 (K), J.2 (Pin_2)
- no-connect marks 0 -> 4
Changed lines of the file:
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@@
 (kicad_sch (version 20220404) (generator eeschema)
   (paper "A4")
-  (symbol_instances)
+  (no_connect (at 128.27 110.49))
+  (no_connect (at 128.27 113.03))
+  (no_connect (at 140.97 113.03))
+  (no_connect (at 140.97 110.49))
+  (wire (pts (xy 160.02 80.01) (xy 160.02 85.09))
+    (stroke (width 0) (type default))
+  )
+  (wire (pts (xy 128.27 107.95) (xy 128.27 92.71))
+    (stroke (width 0) (type default))
+  )
+  (wire (pts (xy 128.27 92.71) (xy 160.02 92.71))
+    (stroke (width 0) (type default))
+  )
+  (wire (pts (xy 160.02 68.58) (xy 160.02 72.39))
+    (stroke (width 0) (type default))
+  )
+  (wire (pts (xy 140.97 107.95) (xy 147.32 107.95))
+    (stroke (width 0) (type default))
+  )
+  (symbol (lib_id "Connector_Generic:Conn_02x03_Odd_Even") (at 133.35 110.49 0) (unit 1)
+    (in_bom yes) (on_board yes) (fields_autoplaced)
+    (default_instance (reference "J") (unit 1) (value "Conn_02x03_Odd_Even") (footprint ""))
+    (property "Reference" "J" (id 0) (at 134.62 102.87 0)
+      (effects (font (size 1.27 1.27)))
+    )
+    (property "Value" "Conn_02x03_Odd_Even" (id 1) (at 134.62 105.41 0)
+      (effects (font (size 1.27 1.27)))
+    )
+    (property "Footprint" "" (id 2) (at 133.35 110.49 0)
+      (effects (font (size 1.27 1.27)) hide)
+    )
+    (property "Datasheet" "~" (id 3) (at 133.35 110.49 0)
+      (effects (font (size 1.27 1.27)) hide)
+    )
+    (pin "1")
+    (pin "2")
+    (pin "3")
+    (pin "4")
+    (pin "5")
+    (pin "6")
+  )
+  (symbol (lib_id "Device:R") (at 160.02 88.9 0) (unit 1)
+    (in_bom yes) (on_board yes) (fields_autoplaced)
+    (default_instance (reference "R") (unit 1) (value "R") (footprint ""))
+    (property "Reference" "R" (id 0) (at 162.56 88.265 0)
+      (effects (font (size 1.27 1.27)) (justify left))
+    )
+    (property "Value" "R" (id 1) (at 162.56 90.805 0)
+      (effects (font (size 1.27 1.27)) (justify left))
+    )
+    (property "Footprint" "" (id 2) (at 158.242 88.9 90)
+      (effects (font (size 1.27 1.27)) hide)
+    )
+    (property "Datasheet" "~" (id 3) (at 160.02 88.9 0)
+      (effects (font (size 1.27 1.27)) hide)
+    )
+    (pin "1")
+    (pin "2")
+  )
+  (symbol (lib_id "power:GND") (at 160.02 68.58 180) (unit 1)
+    (in_bom yes) (on_board yes) (fields_autoplaced)
+    (default_instance (reference "#PWR") (unit 1) (value "GND") (footprint ""))
+    (property "Reference" "#PWR" (id 0) (at 160.02 62.23 0)
+      (effects (font (size 1.27 1.27)) hide)
+    )
+    (property "Value" "GND" (id 1) (at 160.02 64.8437 0)
+      (effects (font (size 1.27 1.27)))
+    )
+    (property "Footprint" "" (id 2) (at 160.02 68.58 0)
+      (effects (font (size 1.27 1.27)) hide)
+    )
+    (property "Datasheet" "" (id 3) (at 160.02 68.58 0)
+      (effects (font (size 1.27 1.27)) hide)
+    )
+    (pin "1")
+  )
+  (symbol (lib_id "Device:LED") (at 160.02 76.2 270) (unit 1)
+    (in_bom yes) (on_board yes) (fields_autoplaced)
+    (default_instance (reference "D") (unit 1) (value "LED") (footprint ""))
+    (property "Reference" "D" (id 0) (at 162.56 73.9775 90)
+      (effects (font (size 1.27 1.27)) (justify left))
+    )
+    (property "Value" "LED" (id 1) (at 162.56 76.5175 90)
+      (effects (font (size 1.27 1.27)) (justify left))
+    )
+    (property "Footprint" "" (id 2) (at 160.02 76.2 0)
+      (effects (font (size 1.27 1.27)) hide)
+    )
+    (property "Datasheet" "~" (id 3) (at 160.02 76.2 0)
+      (effects (font (size 1.27 1.27)) hide)
+    )
+    (pin "1")
+    (pin "2")
+  )
+  (symbol (lib_id "power:GND") (at 147.32 107.95 90) (unit 1)
+    (in_bom yes) (on_board yes) (fields_autoplaced)
+    (default_instance (reference "#PWR") (unit 1) (value "GND") (footprint ""))
+    (property "Reference" "#PWR" (id 0) (at 153.67 107.95 0)
+      (effects (font (size 1.27 1.27)) hide)
+    )
+    (property "Value" "GND" (id 1) (at 151.13 108.585 90)
+      (effects (font (size 1.27 1.27)) (justify right))
+    )
+    (property "Footprint" "" (id 2) (at 147.32 107.95 0)
+      (effects (font (size 1.27 1.27)) hide)
+    )
+    (property "Datasheet" "" (id 3) (at 147.32 107.95 0)
+      (effects (font (size 1.27 1.27)) hide)
+    )
+    (pin "1")
+  )
+  (sheet_instances
+    (path "/" (page "1"))
+  )
+  (symbol_instances
+    (path "/e3bdaf44-d976-49ac-a641-094dd1a8e91b"
+      (reference "#PWR02") (unit 1) (value "GND") (footprint "")
+    )
+    (path "/22f903d9-7725-4505-94cb-1a64b26ee9f9"
+      (reference "#PWR03") (unit 1) (value "GND") (footprint "")
+    )
+    (path "/29ae8e72-4baf-4097-9ddf-52ae73e3903d"
+      (reference "D1") (unit 1) (value "LED") (footprint "sunled:XZDGK45WT-9")
+    )
+    (path "/02b6aad0-aa1d-42ba-9c69-761e9bc4c9e0"
+      (reference "J1") (unit 1) (value "Conn_02x03_Odd_Even") (footprint "Connector_PinHeader_2.54mm:PinHeader_2x03_P2.54mm_Vertical_SMD")
+    )
+    (path "/0ef16558-5163-4725-a2a7-6916b1036929"
+      (reference "R1") (unit 1) (value "R") (footprint "Resistor_SMD:R_1206_3216Metric_Pad1.30x1.75mm_HandSolder")
+    )
+  )
 )
