File: VORTAC_SAO/VORTAC SAO Board.kicad_pcb (KiCad board)
At the start: 2 copper layers, 64.2 x 55.6 mm, 5 parts, among them J1 Simple_Addon_v2, P1 Simple_Addon_v2, P2 Simple_Addon_v2, P3 Simple_Addon_v2

Commit message: added text and credit
Routing:
- added copper zone on B.Cu, net (none)
Other:
- board text added: "@zap!"
- board text added: "Build Inspire Promote"
- board text added: "aerospacevillage.org"
- board text added: "v01"
Changed lines of the file:
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@@
       (xy 171.786543 87.579523)
     ) (layer "User.1") (width 0.1) (fill none))
+  (gr_text "v01" (at 149.86 119.38) (layer "B.Cu")
+    (effects (font (size 1.5 1.5) (thickness 0.3)) (justify mirror))
+  )
+  (gr_text "Build\nInspire\nPromote" (at 140.09641 92.491602) (layer "B.SilkS")
+    (effects (font (size 3 3) (thickness 0.5)) (justify mirror))
+  )
+  (gr_text "@zap!" (at 131.075356 117.163897) (layer "B.SilkS")
+    (effects (font (size 1 1) (thickness 0.15)) (justify mirror))
+  )
+  (gr_text "aerospacevillage.org" (at 139.7 102.87) (layer "B.SilkS")
+    (effects (font (size 2 2) (thickness 0.3)) (justify mirror))
+  )
   (segment (start 139.64 118.09) (end 138.4514 116.9014) (width 0.25) (layer "B.Cu") (net 1))
   (segment (start 120.4976 74.2188) (end 119.0244 75.8952) (width 0.25) (layer "B.Cu") (net 1))
@@
   (segment (start 123.151372 73.7614) (end 119.750798 77.161974) (width 0.25) (layer "F.Cu") (net 6))
   (segment (start 119.634 77.5208) (end 117.7036 78.1304) (width 0.25) (layer "F.Cu") (net 6))
+  (zone (net 0) (net_name "") (layer "B.Cu") (hatch edge 0.508)
+    (connect_pads (clearance 0.508))
+    (min_thickness 0.254) (filled_areas_thickness no)
+    (fill yes (thermal_gap 0.508) (thermal_bridge_width 0.508))
+    (polygon
+      (pts
+        (xy 180.34 60.96)
+        (xy 180.34 130.81)
+        (xy 99.06 130.81)
+        (xy 99.06 59.69)
+      )
+    )
+  )
 )
