File: VORTAC_SAO/VORTAC SAO Board.kicad_pcb (KiCad board)
At the start: 2 copper layers, 64.2 x 55.6 mm, 5 parts, among them J1 Simple_Addon_v2, P1 Simple_Addon_v2, P2 Simple_Addon_v2, P3 Simple_Addon_v2

Commit message: added jlcjlcjlcjlc to the back of the vortac SAO
Other:
- board text added: "jlcjlcjlcjlc"
Changed lines of the file:
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@@
     (effects (font (size 3 3) (thickness 0.5)) (justify mirror))
+  )
+  (gr_text "jlcjlcjlcjlc" (at 159.75 67.05 30) (layer "B.SilkS")
+    (effects (font (size 1 1) (thickness 0.15)) (justify left bottom mirror))
   )
   (gr_text "@zap!" (at 131.075356 117.163897) (layer "B.SilkS")
